Commit message: added navy door test environment

File: robot_model/ground/navy_door.urdf (robot description, URDF)
Before this commit: robot navy_door, 1 links, 0 joints
Links:
- removed link door
- added link door_frame, mass 500.; collision box size=1.4 0.1 0.4; visual mesh filename=package://navy_door_765x1450.stl scale=1 1 1

Commit message: added collisions for side walls to knee-knocker door

File: robot_model/ground/navy_door.urdf (robot description, URDF)
Before this commit: robot navy_door, 1 links, 0 joints
Links:
- link door_frame: mass 500. -> 5000.; geometry collision box size=0.518 0.05 2.2; collision box size=0.518 0.05 2.2
