Commit message: added robot_utils from robotics course and some scripts

File: robot_model/crab/crab.urdf (robot description, URDF)
Before this commit: robot crab_robot, 73 links, 72 joints
Links:
- link back_left__cluster_1_distal_link: geometry collision mesh filename=/home/june/research/PyPnC/robot_model/crab/meshes/776_meshe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; visual mesh filename=/home/june/research/PyPnC/robot_model/crab/meshes/776_meshe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
- link back_left__cluster_1_end_link: geometry collision mesh filename=/home/june/research/PyPnC/robot_model/crab/meshes/776_meshe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; visual mesh filename=/home/june/research/PyPnC/robot_model/crab/meshes/776_meshe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
- link back_left__cluster_1_proximal_link: geometry collision mesh filename=/home/june/research/PyPnC/robot_model/crab/meshes/776_meshe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; visual mesh filename=/home/june/research/PyPnC/robot_model/crab/meshes/776_meshe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
- link back_left__cluster_2_distal_link: geometry collision mesh filename=/home/june/research/PyPnC/robot_model/crab/meshes/665_meshe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; visual mesh filename=/home/june/research/PyPnC/robot_model/crab/meshes/665_meshe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
- link back_left__cluster_2_end_link: geometry collision mesh filename=/home/june/research/PyPnC/robot_model/crab/meshes/665_meshe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; visual mesh filename=/home/june/research/PyPnC/robot_model/crab/meshes/665_meshe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
- link back_left__cluster_2_proximal_link: geometry collision mesh filename=/home/june/research/PyPnC/robot_model/crab/meshes/665_meshe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; visual mesh filename=/home/june/research/PyPnC/robot_model/crab/meshes/665_meshe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
- link back_left__cluster_3_distal_link: geometry collision mesh filename=/home/june/research/PyPnC/robot_model/crab/meshes/5555_mesh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; visual mesh filename=/home/june/research/PyPnC/robot_model/crab/meshes/5555_mesh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
- link back_left__cluster_3_proximal_link: geometry collision mesh filename=/home/june/research/PyPnC/robot_model/crab/meshes/5555_mesh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; visual mesh filename=/home/june/research/PyPnC/robot_model/crab/meshes/5555_mesh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
- link back_left__cluster_3_wrist_link: geometry collision mesh filename=/home/june/research/PyPnC/robot_model/crab/meshes/5555_mesh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; visual mesh filename=/home/june/research/PyPnC/robot_model/crab/meshes/5555_mesh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
- link back_right__cluster_1_distal_link: geometry collision mesh filename=/home/june/research/PyPnC/robot_model/crab/meshes/776_meshe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; visual mesh filename=/home/june/research/PyPnC/robot_model/crab/meshes/776_meshe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
- link back_right__cluster_1_end_link: geometry collision mesh filename=/home/june/research/PyPnC/robot_model/crab/meshes/776_meshe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; visual mesh filename=/home/june/research/PyPnC/robot_model/crab/meshes/776_meshe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
- link back_right__cluster_1_proximal_link: geometry collision mesh filename=/home/june/research/PyPnC/robot_model/crab/meshes/776_meshe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; visual mesh filename=/home/june/research/PyPnC/robot_model/crab/meshes/776_meshe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
- link back_right__cluster_2_distal_link: geometry collision mesh filename=/home/june/research/PyPnC/robot_model/crab/meshes/665_meshe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; visual mesh filename=/home/june/research/PyPnC/robot_model/crab/meshes/665_meshe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
- link back_right__cluster_2_end_link: geometry collision mesh filename=/home/june/research/PyPnC/robot_model/crab/meshes/665_meshe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; visual mesh filename=/home/june/research/PyPnC/robot_model/crab/meshes/665_meshe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
- link back_right__cluster_2_proximal_link: geometry collision mesh filename=/home/june/research/PyPnC/robot_model/crab/meshes/665_meshe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; visual mesh filename=/home/june/research/PyPnC/robot_model/crab/meshes/665_meshe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
- link back_right__cluster_3_distal_link: geometry collision mesh filename=/home/june/research/PyPnC/robot_model/crab/meshes/5555_mesh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; visual mesh filename=/home/june/research/PyPnC/robot_model/crab/meshes/5555_mesh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
- link back_right__cluster_3_proximal_link: geometry collision mesh filename=/home/june/research/PyPnC/robot_model/crab/meshes/5555_mesh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; visual mesh filename=/home/june/research/PyPnC/robot_model/crab/meshes/5555_mesh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
- link back_right__cluster_3_wrist_link: geometry collision mesh filename=/home/june/research/PyPnC/robot_model/crab/meshes/5555_mesh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; visual mesh filename=/home/june/research/PyPnC/robot_model/crab/meshes/5555_mesh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
- link base_link: geometry collision mesh filename=/home/june/research/PyPnC/robot_model/crab/meshes/base_link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 scale=1 1 1; visual mesh filename=/home/june/research/PyPnC/robot_model/crab/meshes/base_link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 scale=1 1 1
- link front_left__cluster_1_distal_link: geometry collision mesh filename=/home/june/research/PyPnC/robot_model/crab/meshes/776_meshe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; visual mesh filename=/home/june/research/PyPnC/robot_model/crab/meshes/776_meshe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
- link front_left__cluster_1_end_link: geometry collision mesh filename=/home/june/research/PyPnC/robot_model/crab/meshes/776_meshe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; visual mesh filename=/home/june/research/PyPnC/robot_model/crab/meshes/776_meshe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
- link front_left__cluster_1_proximal_link: geometry collision mesh filename=/home/june/research/PyPnC/robot_model/crab/meshes/776_meshe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; visual mesh filename=/home/june/research/PyPnC/robot_model/crab/meshes/776_meshe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
- link front_left__cluster_2_distal_link: geometry collision mesh filename=/home/june/research/PyPnC/robot_model/crab/meshes/665_meshe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; visual mesh filename=/home/june/research/PyPnC/robot_model/crab/meshes/665_meshe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
- link front_left__cluster_2_end_link: geometry collision mesh filename=/home/june/research/PyPnC/robot_model/crab/meshes/665_meshe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; visual mesh filename=/home/june/research/PyPnC/robot_model/crab/meshes/665_meshe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
- link front_left__cluster_2_proximal_link: geometry collision mesh filename=/home/june/research/PyPnC/robot_model/crab/meshes/665_meshe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; visual mesh filename=/home/june/research/PyPnC/robot_model/crab/meshes/665_meshe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
- link front_left__cluster_3_distal_link: geometry collision mesh filename=/home/june/research/PyPnC/robot_model/crab/meshes/5555_mesh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; visual mesh filename=/home/june/research/PyPnC/robot_model/crab/meshes/5555_mesh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
- link front_left__cluster_3_proximal_link: geometry collision mesh filename=/home/june/research/PyPnC/robot_model/crab/meshes/5555_mesh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; visual mesh filename=/home/june/research/PyPnC/robot_model/crab/meshes/5555_mesh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
- link front_left__cluster_3_wrist_link: geometry collision mesh filename=/home/june/research/PyPnC/robot_model/crab/meshes/5555_mesh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; visual mesh filename=/home/june/research/PyPnC/robot_model/crab/meshes/5555_mesh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
- link front_right__cluster_1_distal_link: geometry collision mesh filename=/home/june/research/PyPnC/robot_model/crab/meshes/776_meshe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; visual mesh filename=/home/june/research/PyPnC/robot_model/crab/meshes/776_meshe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
- link front_right__cluster_1_end_link: geometry collision mesh filename=/home/june/research/PyPnC/robot_model/crab/meshes/776_meshe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; visual mesh filename=/home/june/research/PyPnC/robot_model/crab/meshes/776_meshe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
- link front_right__cluster_1_proximal_link: geometry collision mesh filename=/home/june/research/PyPnC/robot_model/crab/meshes/776_meshe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; visual mesh filename=/home/june/research/PyPnC/robot_model/crab/meshes/776_meshe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
- link front_right__cluster_2_distal_link: geometry collision mesh filename=/home/june/research/PyPnC/robot_model/crab/meshes/665_meshe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; visual mesh filename=/home/june/research/PyPnC/robot_model/crab/meshes/665_meshe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
- link front_right__cluster_2_end_link: geometry collision mesh filename=/home/june/research/PyPnC/robot_model/crab/meshes/665_meshe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; visual mesh filename=/home/june/research/PyPnC/robot_model/crab/meshes/665_meshe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
- link front_right__cluster_2_proximal_link: geometry collision mesh filename=/home/june/research/PyPnC/robot_model/crab/meshes/665_meshe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; visual mesh filename=/home/june/research/PyPnC/robot_model/crab/meshes/665_meshe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
- link front_right__cluster_3_distal_link: geometry collision mesh filename=/home/june/research/PyPnC/robot_model/crab/meshes/5555_mesh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; visual mesh filename=/home/june/research/PyPnC/robot_model/crab/meshes/5555_mesh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
- link front_right__cluster_3_proximal_link: geometry collision mesh filename=/home/june/research/PyPnC/robot_model/crab/meshes/5555_mesh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; visual mesh filename=/home/june/research/PyPnC/robot_model/crab/meshes/5555_mesh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
- link front_right__cluster_3_wrist_link: geometry collision mesh filename=/home/june/research/PyPnC/robot_model/crab/meshes/5555_mesh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; visual mesh filename=/home/june/research/PyPnC/robot_model/crab/meshes/5555_mesh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
