Commit message: got ergoCub step on knee knocker behavior working with SCA
changes:
* added offset from floating base to torso link used for frame planning
* remove default collisions in ergoCub URDF for primitive geometry
* fixed usage of normal plane in contact
* uses casadi only when using Self Collsion Avoidance (SCA)
* adds unit test for ergoCub stepping on knee knocker w/o and w/ SCA
* fixed IRIS sequence routine when > 3 IRIS regions, apply it only when
overlapping regions exist

File: robot_model/ergoCub/ergoCub.urdf (robot description, URDF)
Before this commit: robot ergoCub, 204 links, 203 joints
Links:
- added link torso_primitive_shape, mass 1e-9; collision box size=0.18 0.27 0.6
- link chest: geometry visual mesh filename=package://meshes/simmechanics/sim_ecub_1-1_chest.stl scale=0.001 0.001 0.001
- link head: geometry visual mesh filename=package://meshes/simmechanics/sim_ecub_1-1_head.stl scale=0.001 0.001 0.001
- link l_ankle_1: geometry visual mesh filename=package://meshes/simmechanics/sim_ecub_1-1_l_ankle_1.stl scale=0.001 0.001 0.001
- link l_ankle_2: geometry visual mesh filename=package://meshes/simmechanics/sim_ecub_1-1_l_ankle_2.stl scale=0.001 0.001 0.001
- link l_foot_front: geometry visual mesh filename=package://meshes/simmechanics/sim_ecub_1-1_l_foot_front.stl scale=0.001 0.001 0.001
- link l_foot_rear: geometry visual mesh filename=package://meshes/simmechanics/sim_ecub_1-1_l_foot_rear.stl scale=0.001 0.001 0.001
- link l_forearm: geometry visual mesh filename=package://meshes/simmechanics/sim_ecub_1-1_l_forearm.stl scale=0.001 0.001 0.001
- link l_hand_index_1: geometry visual mesh filename=package://meshes/simmechanics/sim_ecub_1-1_l_hand_index_1.s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 scale=0.001 0.001 0.001
- link l_hand_index_2: geometry visual mesh filename=package://meshes/simmechanics/sim_ecub_1-1_l_hand_index_2.s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 scale=0.001 0.001 0.001
- link l_hand_index_3: geometry visual mesh filename=package://meshes/simmechanics/sim_ecub_1-1_l_hand_index_3.s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 scale=0.001 0.001 0.001
- link l_hand_middle_1: geometry visual mesh filename=package://meshes/simmechanics/sim_ecub_1-1_l_hand_middle_1.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 scale=0.001 0.001 0.001
- link l_hand_middle_2: geometry visual mesh filename=package://meshes/simmechanics/sim_ecub_1-1_l_hand_middle_2.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 scale=0.001 0.001 0.001
- link l_hand_palm: geometry collision sphere radius=0.03; visual mesh filename=package://meshes/simmechanics/sim_ecub_1-1_l_hand_palm.stl scale=0.001 0.001 0.001
- link l_hand_pinkie_1: geometry visual mesh filename=package://meshes/simmechanics/sim_ecub_1-1_l_hand_pinkie_1.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 scale=0.001 0.001 0.001
- link l_hand_pinkie_2: geometry visual mesh filename=package://meshes/simmechanics/sim_ecub_1-1_l_hand_pinkie_2.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 scale=0.001 0.001 0.001
- link l_hand_ring_1: geometry visual mesh filename=package://meshes/simmechanics/sim_ecub_1-1_l_hand_ring_1.stl scale=0.001 0.001 0.001
- link l_hand_ring_2: geometry visual mesh filename=package://meshes/simmechanics/sim_ecub_1-1_l_hand_ring_2.stl scale=0.001 0.001 0.001
- link l_hand_thumb_1: geometry visual mesh filename=package://meshes/simmechanics/sim_ecub_1-1_l_hand_thumb_1.s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 scale=0.001 0.001 0.001
- link l_hand_thumb_2: geometry visual mesh filename=package://meshes/simmechanics/sim_ecub_1-1_l_hand_thumb_2.s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 scale=0.001 0.001 0.001
- link l_hand_thumb_3: geometry visual mesh filename=package://meshes/simmechanics/sim_ecub_1-1_l_hand_thumb_3.s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 scale=0.001 0.001 0.001
- link l_hip_1: geometry visual mesh filename=package://meshes/simmechanics/sim_ecub_1-1_l_hip_1.stl scale=0.001 0.001 0.001
- link l_hip_2: geometry visual mesh filename=package://meshes/simmechanics/sim_ecub_1-1_l_hip_2.stl scale=0.001 0.001 0.001
- link l_hip_3: geometry visual mesh filename=package://meshes/simmechanics/sim_ecub_1-1_l_hip_3.stl scale=0.001 0.001 0.001
- link l_lower_leg: geometry collision sphere radius=0.05; visual mesh filename=package://meshes/simmechanics/sim_ecub_1-1_l_lower_leg.stl scale=0.001 0.001 0.001
- link l_shoulder_1: geometry visual mesh filename=package://meshes/simmechanics/sim_ecub_1-1_l_shoulder_1.stl scale=0.001 0.001 0.001
- link l_shoulder_2: geometry visual mesh filename=package://meshes/simmechanics/sim_ecub_1-1_l_shoulder_2.stl scale=0.001 0.001 0.001
- link l_shoulder_3: geometry visual mesh filename=package://meshes/simmechanics/sim_ecub_1-1_l_shoulder_3.stl scale=0.001 0.001 0.001
- link l_upper_arm: geometry visual mesh filename=package://meshes/simmechanics/sim_ecub_1-1_l_upperarm.stl scale=0.001 0.001 0.001
- link l_upper_leg: geometry visual mesh filename=package://meshes/simmechanics/sim_ecub_1-1_l_upper_leg.stl scale=0.001 0.001 0.001
- link l_wrist_1: geometry visual mesh filename=package://meshes/simmechanics/sim_ecub_1-1_l_wrist_1.stl scale=0.001 0.001 0.001
- link l_wrist_2: geometry visual mesh filename=package://meshes/simmechanics/sim_ecub_1-1_l_wrist_2.stl scale=0.001 0.001 0.001
- link neck_2: geometry visual mesh filename=package://meshes/simmechanics/sim_ecub_1-1_head_neck_2.stl scale=0.001 0.001 0.001
- link neck_3: geometry visual mesh filename=package://meshes/simmechanics/sim_ecub_1-1_head_neck_3.stl scale=0.001 0.001 0.001
- link r_ankle_1: geometry visual mesh filename=package://meshes/simmechanics/sim_ecub_1-1_r_ankle_1.stl scale=0.001 0.001 0.001
- link r_ankle_2: geometry visual mesh filename=package://meshes/simmechanics/sim_ecub_1-1_r_ankle_2.stl scale=0.001 0.001 0.001
- link r_foot_front: geometry visual mesh filename=package://meshes/simmechanics/sim_ecub_1-1_r_foot_front.stl scale=0.001 0.001 0.001
- link r_foot_rear: geometry visual mesh filename=package://meshes/simmechanics/sim_ecub_1-1_r_foot_rear.stl scale=0.001 0.001 0.001
- link r_forearm: geometry visual mesh filename=package://meshes/simmechanics/sim_ecub_1-1_r_forearm.stl scale=0.001 0.001 0.001
- link r_hand_index_1: geometry visual mesh filename=package://meshes/simmechanics/sim_ecub_1-1_r_hand_index_1.s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 scale=0.001 0.001 0.001
- link r_hand_index_2: geometry visual mesh filename=package://meshes/simmechanics/sim_ecub_1-1_r_hand_index_2.s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 scale=0.001 0.001 0.001
- link r_hand_index_3: geometry visual mesh filename=package://meshes/simmechanics/sim_ecub_1-1_r_hand_index_3.s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 scale=0.001 0.001 0.001
- link r_hand_middle_1: geometry visual mesh filename=package://meshes/simmechanics/sim_ecub_1-1_r_hand_middle_1.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 scale=0.001 0.001 0.001
- link r_hand_middle_2: geometry visual mesh filename=package://meshes/simmechanics/sim_ecub_1-1_r_hand_middle_2.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 scale=0.001 0.001 0.001
- link r_hand_palm: geometry collision sphere radius=0.03; visual mesh filename=package://meshes/simmechanics/sim_ecub_1-1_r_hand_palm.stl scale=0.001 0.001 0.001
- link r_hand_pinkie_1: geometry visual mesh filename=package://meshes/simmechanics/sim_ecub_1-1_r_hand_pinkie_1.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 scale=0.001 0.001 0.001
- link r_hand_pinkie_2: geometry visual mesh filename=package://meshes/simmechanics/sim_ecub_1-1_r_hand_pinkie_2.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 scale=0.001 0.001 0.001
- link r_hand_ring_1: geometry visual mesh filename=package://meshes/simmechanics/sim_ecub_1-1_r_hand_ring_1.stl scale=0.001 0.001 0.001
- link r_hand_ring_2: geometry visual mesh filename=package://meshes/simmechanics/sim_ecub_1-1_r_hand_ring_2.stl scale=0.001 0.001 0.001
- link r_hand_thumb_1: geometry visual mesh filename=package://meshes/simmechanics/sim_ecub_1-1_r_hand_thumb_1.s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 scale=0.001 0.001 0.001
- link r_hand_thumb_2: geometry visual mesh filename=package://meshes/simmechanics/sim_ecub_1-1_r_hand_thumb_2.s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 scale=0.001 0.001 0.001
- link r_hand_thumb_3: geometry visual mesh filename=package://meshes/simmechanics/sim_ecub_1-1_r_hand_thumb_3.s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 scale=0.001 0.001 0.001
- link r_hip_1: geometry visual mesh filename=package://meshes/simmechanics/sim_ecub_1-1_r_hip_1.stl scale=0.001 0.001 0.001
- link r_hip_2: geometry visual mesh filename=package://meshes/simmechanics/sim_ecub_1-1_r_hip_2.stl scale=0.001 0.001 0.001
- link r_hip_3: geometry visual mesh filename=package://meshes/simmechanics/sim_ecub_1-1_r_hip_3.stl scale=0.001 0.001 0.001
- link r_lower_leg: geometry collision sphere radius=0.05; visual mesh filename=package://meshes/simmechanics/sim_ecub_1-1_r_lower_leg.stl scale=0.001 0.001 0.001
- link r_shoulder_1: geometry visual mesh filename=package://meshes/simmechanics/sim_ecub_1-1_r_shoulder_1.stl scale=0.001 0.001 0.001
- link r_shoulder_2: geometry visual mesh filename=package://meshes/simmechanics/sim_ecub_1-1_r_shoulder_2.stl scale=0.001 0.001 0.001
- link r_shoulder_3: geometry visual mesh filename=package://meshes/simmechanics/sim_ecub_1-1_r_shoulder_3.stl scale=0.001 0.001 0.001
- link r_upper_arm: geometry visual mesh filename=package://meshes/simmechanics/sim_ecub_1-1_r_upperarm.stl scale=0.001 0.001 0.001
- link r_upper_leg: geometry visual mesh filename=package://meshes/simmechanics/sim_ecub_1-1_r_upper_leg.stl scale=0.001 0.001 0.001
- link r_wrist_1: geometry visual mesh filename=package://meshes/simmechanics/sim_ecub_1-1_r_wrist_1.stl scale=0.001 0.001 0.001
- link r_wrist_2: geometry visual mesh filename=package://meshes/simmechanics/sim_ecub_1-1_r_wrist_2.stl scale=0.001 0.001 0.001
- link realsense: geometry visual mesh filename=package://meshes/simmechanics/sim_ecub_1-1_realsense.stl scale=0.001 0.001 0.001
- link root_link: geometry visual mesh filename=package://meshes/simmechanics/sim_ecub_1-1_root_link.stl scale=0.001 0.001 0.001
- link torso_1: geometry visual mesh filename=package://meshes/simmechanics/sim_ecub_1-1_torso_1.stl scale=0.001 0.001 0.001
- link torso_2: geometry visual mesh filename=package://meshes/simmechanics/sim_ecub_1-1_torso_2.stl scale=0.001 0.001 0.001
Joints:
- added joint torso_primitive_shape_joint: type fixed, parent root_link, child torso_primitive_shape, origin xyz=0.0 0.0 0.3 rpy=0 0 0
- joint l_hand_thumb_skin_1_fixed_joint: origin xyz=0.028280418005286963 -0.0031311476143920103 0.0033000000000000806 rpy=-1.5707963267948961 -7.216449660063518e-16 -2.1816615649914324 -> xyz=0.028280418005286963 -0.0031311476143919548 0.0033000000000000806 rpy=-1.5707963267948961 -7.216449660063518e-16 -2.1816615649914324

Commit message: generates SCA and full-body motion for ergoCub stepping on knee knocker for ErgoCub
changes include:
* changes default collusions for box-sphere collisions
* re-factoring ErgoCubMulticontactPlanner to allow for contact phase
speed ups
* gain tunning on full-body TO (speed up phase currently hard-coded)
* adds kinematic reachability of knees
* temperarily removes usage of set_contact_breaking_velocity to use
CLARABEL solver

File: robot_model/ergoCub/ergoCub.urdf (robot description, URDF)
Before this commit: robot ergoCub, 205 links, 204 joints
Links:
- link l_hand_palm: geometry visual mesh filename=package://meshes/simmechanics/sim_ecub_1-1_l_hand_palm.stl scale=0.001 0.001 0.001
Joints:
- joint l_index_add: axis 1.1895336853461886e-15 0.9999999999999999 -1.9812040713213337e-15 -> (none); limit lower=0 upper=0.2617993877991494 effort=1e+9 velocity=1e+9 -> (none); type revolute -> fixed
- joint l_index_dist: axis -1 -2.359224176539984e-16 4.163337069211178e-17 -> (none); limit lower=0 upper=1.7994344588061537 effort=1e+9 velocity=1e+9 -> (none); type revolute -> fixed
- joint l_index_prox: axis -1 8.326672684688522e-17 7.023654435833748e-10 -> (none); limit lower=0 upper=1.5707963267948966 effort=1e+9 velocity=1e+9 -> (none); type revolute -> fixed
- joint l_middle_dist: axis -1 1.952334931070572e-12 1.0795870667149422e-10 -> (none); limit lower=0 upper=1.7994344588061537 effort=1e+9 velocity=1e+9 -> (none); type revolute -> fixed
- joint l_middle_prox: axis -1.0000000000000004 1.6098145522958664e-16 4.176883423103147e-15 -> (none); limit lower=0 upper=1.5707963267948966 effort=1e+9 velocity=1e+9 -> (none); type revolute -> fixed
- joint l_pinkie_dist: axis -0.9999999998538309 7.645451042193251e-6 -1.5293310428212298e-5 -> (none); limit lower=0 upper=1.7226399717184033 effort=1e+9 velocity=1e+9 -> (none); type revolute -> fixed
- joint l_pinkie_prox: axis -0.9999999998538295 7.644772463726695e-6 -1.529375771042174e-5 -> (none); limit lower=0 upper=1.5707963267948966 effort=1e+9 velocity=1e+9 -> (none); type revolute -> fixed
- joint l_ring_dist: axis -1 -2.617159685310911e-13 1.0794249544288393e-10 -> (none); limit lower=0 upper=1.7994344588061537 effort=1e+9 velocity=1e+9 -> (none); type revolute -> fixed
- joint l_ring_prox: axis -1.0000000000000002 4.364549018964596e-17 3.6637359812630166e-15 -> (none); limit lower=0 upper=1.5707963267948966 effort=1e+9 velocity=1e+9 -> (none); type revolute -> fixed
- joint l_thumb_add: axis 9.71445146547012e-16 1.0269562977782698e-15 -1.0000000000000002 -> (none); limit lower=0 upper=1.7453292519943295 effort=1e+9 velocity=1e+9 -> (none); type revolute -> fixed
- joint l_thumb_dist: axis -1.846719305254041e-11 -1.8750709318560158e-11 -0.9999999999999996 -> (none); limit lower=0 upper=1.7697638615222502 effort=1e+9 velocity=1e+9 -> (none); type revolute -> fixed
- joint l_thumb_prox: axis 5.134781488891349e-16 3.1363800445660672e-15 -0.9999999999999996 -> (none); limit lower=0 upper=1.5707963267948966 effort=1e+9 velocity=1e+9 -> (none); type revolute -> fixed
- joint r_index_add: axis -5.389323627044831e-16 -0.9999999999999999 1.6046911875538946e-15 -> (none); limit lower=0 upper=0.2617993877991494 effort=1e+9 velocity=1e+9 -> (none); type revolute -> fixed
- joint r_index_dist: axis -0.9999999999999993 -2.0122792321330975e-16 -4.510281037539697e-16 -> (none); limit lower=0 upper=1.7994344588061537 effort=1e+9 velocity=1e+9 -> (none); type revolute -> fixed
- joint r_index_prox: axis -0.9999999999999993 3.434752482434078e-15 -1.672273430841644e-15 -> (none); limit lower=0 upper=1.5707963267948966 effort=1e+9 velocity=1e+9 -> (none); type revolute -> fixed
- joint r_middle_dist: axis -0.9999999999999998 -2.0695253452753748e-15 -1.0792969296086812e-10 -> (none); limit lower=0 upper=1.7994344588061537 effort=1e+9 velocity=1e+9 -> (none); type revolute -> fixed
- joint r_middle_prox: axis -0.9999999999999996 -4.562322741819007e-15 1.079337105802658e-10 -> (none); limit lower=0 upper=1.5707963267948966 effort=1e+9 velocity=1e+9 -> (none); type revolute -> fixed
- joint r_pinkie_dist: axis -0.9999999999999999 9.036247971209683e-16 -2.4586692098222613e-15 -> (none); limit lower=0 upper=1.7226399717184033 effort=1e+9 velocity=1e+9 -> (none); type revolute -> fixed
- joint r_pinkie_prox: axis -0.9999999999999998 4.364801434782878e-15 0 -> (none); limit lower=0 upper=1.5707963267948966 effort=1e+9 velocity=1e+9 -> (none); type revolute -> fixed
- joint r_ring_dist: axis -0.9999999999999999 2.4672971998818127e-13 -1.0789569585001324e-10 -> (none); limit lower=0 upper=1.7994344588061537 effort=1e+9 velocity=1e+9 -> (none); type revolute -> fixed
- joint r_ring_prox: axis -0.9999999999999997 -2.498435601042699e-13 1.0789123761067998e-10 -> (none); limit lower=0 upper=1.5707963267948966 effort=1e+9 velocity=1e+9 -> (none); type revolute -> fixed
- joint r_thumb_add: axis -1.0793213545134961e-10 2.4089270891491094e-15 0.9999999999999998 -> (none); limit lower=0 upper=1.7453292519943295 effort=1e+9 velocity=1e+9 -> (none); type revolute -> fixed
- joint r_thumb_dist: axis 1.8458673825549887e-11 1.8743298579870785e-11 -0.9999999999999999 -> (none); limit lower=0 upper=1.7697638615222502 effort=1e+9 velocity=1e+9 -> (none); type revolute -> fixed
- joint r_thumb_prox: axis 9.992007221626409e-16 -1.1102230246251565e-15 -0.9999999999999997 -> (none); limit lower=0 upper=1.5707963267948966 effort=1e+9 velocity=1e+9 -> (none); type revolute -> fixed

Commit message: remove camera_tilt DoF as it's not needed for multicontact planning

File: robot_model/ergoCub/ergoCub.urdf (robot description, URDF)
Before this commit: robot ergoCub, 205 links, 204 joints
Joints:
- joint camera_tilt: limit lower=-0.5235987755982988 upper=0.5235987755982988 effort=1e+9 velocity=1e+9 -> (none); type revolute -> fixed

Commit message: checked ergoCub plans run on hole in wall and tilted stairs

File: robot_model/ergoCub/ergoCub.urdf (robot description, URDF)
Before this commit: robot ergoCub, 205 links, 204 joints
Links:
- link l_hand_palm: geometry collision sphere radius=0.03; visual mesh filename=package://meshes/simmechanics/sim_ecub_1-1_l_hand_palm.stl scale=0.001 0.001 0.001
Joints:
- joint l_ankle_roll: limit lower=-0.4363323129985824 upper=0.4363323129985824 effort=1e+9 velocity=1e+9 -> lower=-0.63 upper=0.63 effort=1e+9 velocity=1e+9
- joint r_ankle_roll: limit lower=-0.4363323129985824 upper=0.4363323129985824 effort=1e+9 velocity=1e+9 -> lower=-0.63 upper=0.63 effort=1e+9 velocity=1e+9
