Commit message: added urdf with cylinders, spheres, and box collisions

File: robot_model/g1_description/g1_29dof_simple_collisions.urdf (robot description, URDF)
Before this commit: robot g1_29dof_lock_waist, 41 links, 40 joints
Links:
- link left_hip_roll_link: geometry collision cylinder length=0.22 radius=0.05; visual mesh filename=meshes/left_hip_roll_link.STL
- link left_knee_link: geometry collision cylinder length=0.26 radius=0.05; visual mesh filename=meshes/left_knee_link.STL
- link right_hip_roll_link: geometry collision cylinder length=0.22 radius=0.05; visual mesh filename=meshes/right_hip_roll_link.STL
- link right_knee_link: geometry collision cylinder length=0.26 radius=0.05; visual mesh filename=meshes/right_knee_link.STL

Commit message: added SCA refinement with SQP solver option
also fixed plotting plotting from correct fddp solver and adding
extended RoM to G1 ankle roll on simple_collisions URDF model

File: robot_model/g1_description/g1_29dof_simple_collisions.urdf (robot description, URDF)
Before this commit: robot g1_29dof_lock_waist, 41 links, 40 joints
Joints:
- joint left_ankle_roll_joint: limit lower=-0.2618 upper=0.2618 effort=35 velocity=30 -> lower=-0.63 upper=0.63 effort=35 velocity=30
- joint right_ankle_roll_joint: limit lower=-0.2618 upper=0.2618 effort=35 velocity=30 -> lower=-0.63 upper=0.63 effort=35 velocity=30

Commit message: added upper body simplified collisions to G1

File: robot_model/g1_description/g1_29dof_simple_collisions.urdf (robot description, URDF)
Before this commit: robot g1_29dof_lock_waist, 41 links, 40 joints
Links:
- link left_elbow_link: geometry collision cylinder length=0.12 radius=0.035; visual mesh filename=meshes/left_elbow_link.STL
- link left_shoulder_yaw_link: geometry collision cylinder length=0.15 radius=0.03; visual mesh filename=meshes/left_shoulder_yaw_link.STL
- link right_elbow_link: geometry collision cylinder length=0.12 radius=0.035; visual mesh filename=meshes/right_elbow_link.STL
- link right_shoulder_yaw_link: geometry collision cylinder length=0.15 radius=0.03; visual mesh filename=meshes/right_shoulder_yaw_link.STL
- link torso_primitive_shape: geometry collision box size=0.14 0.20 0.45

Commit message: create all cylinder collisions

File: robot_model/g1_description/g1_29dof_simple_collisions.urdf (robot description, URDF)
Before this commit: robot g1_29dof_lock_waist, 41 links, 40 joints
Links:
- link left_ankle_roll_link: geometry collision cylinder length=0.21 radius=0.04; visual mesh filename=meshes/left_ankle_roll_link.STL
- link left_hip_roll_link: geometry collision cylinder length=0.28 radius=0.06; visual mesh filename=meshes/left_hip_roll_link.STL
- link left_knee_link: geometry collision cylinder length=0.3 radius=0.06; visual mesh filename=meshes/left_knee_link.STL
- link left_wrist_roll_link: geometry collision sphere radius=0.035; visual mesh filename=meshes/left_wrist_roll_link.STL
- link right_ankle_roll_link: geometry collision cylinder length=0.21 radius=0.04; visual mesh filename=meshes/right_ankle_roll_link.STL
- link right_hip_roll_link: geometry collision cylinder length=0.28 radius=0.06; visual mesh filename=meshes/right_hip_roll_link.STL
- link right_knee_link: geometry collision cylinder length=0.3 radius=0.06; visual mesh filename=meshes/right_knee_link.STL
- link right_wrist_roll_link: geometry collision sphere radius=0.035; visual mesh filename=meshes/right_wrist_roll_link.STL
- link torso_primitive_shape: geometry collision cylinder length=0.1 radius=0.08; collision cylinder length=0.35 radius=0.11
Joints:
- joint torso_primitive_shape_joint: origin xyz=0 0 0.2 rpy=0 0 0 -> xyz=0 0 0.19 rpy=0 0 0
