Commit message: created and added convex hull of G1 knee for collision check stats
also added the stairs environment, which could use some cleanup

File: robot_model/g1_description/g1_29dof_lock_waist_chull.urdf (robot description, URDF)
Before this commit: robot g1_29dof_lock_waist, 39 links, 38 joints
Links:
- link left_knee_link: geometry collision mesh filename=meshes/left_knee_link_chull.STL; visual mesh filename=meshes/left_knee_link.STL
- link right_knee_link: geometry collision mesh filename=meshes/right_knee_link_chull.STL; visual mesh filename=meshes/right_knee_link.STL

Commit message: include mfpp into collision plots
also added convex hull of pelvis_contour

File: robot_model/g1_description/g1_29dof_lock_waist_chull.urdf (robot description, URDF)
Before this commit: robot g1_29dof_lock_waist, 39 links, 38 joints
Links:
- link pelvis_contour_link: geometry collision mesh filename=meshes/pelvis_contour_link_chull.STL; visual mesh filename=meshes/pelvis_contour_link.STL

Commit message: print collision distances in mm
also added pelvis_contour chull

File: robot_model/g1_description/g1_29dof_lock_waist_chull.urdf (robot description, URDF)
Before this commit: robot g1_29dof_lock_waist, 39 links, 38 joints
Links:
- link right_shoulder_yaw_link: geometry collision mesh filename=meshes/right_shoulder_yaw_link_chull.STL; visual mesh filename=meshes/right_shoulder_yaw_link.STL
