Commit message: fixed SCA to use safe point list
also added recording of resulting CoM and actual frame positions to pkl
file

File: robot_model/g1_description/g1_29dof_lock_waist_modified.urdf (robot description, URDF)
Before this commit: robot g1_29dof_lock_waist, 40 links, 39 joints
Links:
- link left_ankle_roll_link: geometry collision sphere radius=0.025; visual mesh filename=meshes/left_ankle_roll_link.STL
- link right_ankle_roll_link: geometry collision sphere radius=0.025; visual mesh filename=meshes/right_ankle_roll_link.STL
- link torso_link: geometry collision box size=0.14 0.21 0.45; visual mesh filename=meshes/torso_link.STL

Commit message: fixed saving costs, contact orientation so that friction is identity, and torso_primitive in g1 urdf

File: robot_model/g1_description/g1_29dof_lock_waist_modified.urdf (robot description, URDF)
Before this commit: robot g1_29dof_lock_waist, 40 links, 39 joints
Links:
- added link torso_primitive_shape, mass 1e-9; collision box size=0.14 0.31 0.45
- link left_ankle_roll_link: geometry visual mesh filename=meshes/left_ankle_roll_link.STL
- link left_rubber_hand: geometry collision sphere radius=0.035; visual mesh filename=meshes/left_rubber_hand.STL
- link right_ankle_roll_link: geometry visual mesh filename=meshes/right_ankle_roll_link.STL
- link right_rubber_hand: geometry collision sphere radius=0.035; visual mesh filename=meshes/right_rubber_hand.STL
- link torso_link: geometry visual mesh filename=meshes/torso_link.STL
Joints:
- added joint torso_primitive_shape_joint: type fixed, parent pelvis, child torso_primitive_shape, origin xyz=0 0 0.2 rpy=0 0 0

Commit message: wip adding modular quasi-static initial guess

File: robot_model/g1_description/g1_29dof_lock_waist_modified.urdf (robot description, URDF)
Before this commit: robot g1_29dof_lock_waist, 41 links, 40 joints
Links:
- link left_rubber_hand: geometry visual mesh filename=meshes/left_rubber_hand.STL
- link right_rubber_hand: geometry visual mesh filename=meshes/right_rubber_hand.STL

Commit message: tuning for G1 on door contact sequence 1
also added jvel penalty on joints of contacting limbs during
FinalActionModel

File: robot_model/g1_description/g1_29dof_lock_waist_modified.urdf (robot description, URDF)
Before this commit: robot g1_29dof_lock_waist, 41 links, 40 joints
Links:
- link left_ankle_roll_link: geometry collision sphere radius=0.04; visual mesh filename=meshes/left_ankle_roll_link.STL
- link left_rubber_hand: geometry collision sphere radius=0.035; visual mesh filename=meshes/left_rubber_hand.STL
- link right_ankle_roll_link: geometry collision sphere radius=0.04; visual mesh filename=meshes/right_ankle_roll_link.STL
- link right_rubber_hand: geometry collision sphere radius=0.035; visual mesh filename=meshes/right_rubber_hand.STL
Joints:
- joint torso_primitive_shape_joint: parent pelvis -> torso_link

Commit message: added debugging dual vars indices, fixed order of lagr mult guess, fixed feet rotations, and roll limits

File: robot_model/g1_description/g1_29dof_lock_waist_modified.urdf (robot description, URDF)
Before this commit: robot g1_29dof_lock_waist, 41 links, 40 joints
Joints:
- joint left_ankle_roll_joint: limit lower=-0.2618 upper=0.2618 effort=35 velocity=30 -> lower=-0.6284 upper=0.6284 effort=35 velocity=30
- joint right_ankle_roll_joint: limit lower=-0.2618 upper=0.2618 effort=35 velocity=30 -> lower=-0.6284 upper=0.6284 effort=35 velocity=30

Commit message: added clearance to tilted stairs steps

File: robot_model/g1_description/g1_29dof_lock_waist_modified.urdf (robot description, URDF)
Before this commit: robot g1_29dof_lock_waist, 41 links, 40 joints
Joints:
- joint left_ankle_roll_joint: limit lower=-0.6284 upper=0.6284 effort=35 velocity=30 -> lower=-0.63 upper=0.63 effort=35 velocity=30
- joint right_ankle_roll_joint: limit lower=-0.6284 upper=0.6284 effort=35 velocity=30 -> lower=-0.63 upper=0.63 effort=35 velocity=30

Commit message: tuning G1 after adding higher cost on reference for contact jpos / jvel

File: robot_model/g1_description/g1_29dof_lock_waist_modified.urdf (robot description, URDF)
Before this commit: robot g1_29dof_lock_waist, 41 links, 40 joints
Links:
- link left_knee_link: geometry collision sphere radius=0.08; visual mesh filename=meshes/left_knee_link.STL
- link right_knee_link: geometry collision sphere radius=0.08; visual mesh filename=meshes/right_knee_link.STL
- link torso_primitive_shape: geometry collision box size=0.20 0.31 0.50

Commit message: switched collisions to capsules

File: robot_model/g1_description/g1_29dof_lock_waist_modified.urdf (robot description, URDF)
Before this commit: robot g1_29dof_lock_waist, 41 links, 40 joints
Joints:
- joint torso_primitive_shape_joint: origin xyz=0 0 0.2 rpy=0 0 0 -> xyz=0 0 0.15 rpy=0 0 0

File: robot_model/g1_description/g1_29dof_simple_collisions.urdf (robot description, URDF)
Before this commit: robot g1_29dof_lock_waist, 41 links, 40 joints
Links:
- link left_ankle_roll_link: geometry collision cylinder length=0.18 radius=0.035; visual mesh filename=meshes/left_ankle_roll_link.STL
- link left_hip_roll_link: geometry collision cylinder length=0.2 radius=0.06; visual mesh filename=meshes/left_hip_roll_link.STL
- link right_ankle_roll_link: geometry collision cylinder length=0.18 radius=0.035; visual mesh filename=meshes/right_ankle_roll_link.STL
- link right_hip_roll_link: geometry collision cylinder length=0.2 radius=0.06; visual mesh filename=meshes/right_hip_roll_link.STL
- link torso_primitive_shape: geometry collision cylinder length=0.32 radius=0.11
Joints:
- joint torso_primitive_shape_joint: origin xyz=0 0 0.19 rpy=0 0 0 -> xyz=0 0 0.21 rpy=0 0 0

Commit message: tuning for door demos

File: robot_model/g1_description/g1_29dof_lock_waist_modified.urdf (robot description, URDF)
Before this commit: robot g1_29dof_lock_waist, 41 links, 40 joints
Joints:
- joint torso_primitive_shape_joint: origin xyz=0 0 0.15 rpy=0 0 0 -> xyz=0 0 0.2 rpy=0 0 0

Commit message: minor tuning changes
* created bigger box dimensions for kin planner
* changed ipopt optim mu_strategy to adaptive with larger J_reg
* saved weights used in plans

File: robot_model/g1_description/g1_29dof_lock_waist_modified.urdf (robot description, URDF)
Before this commit: robot g1_29dof_lock_waist, 41 links, 40 joints
Links:
- link left_rubber_hand: geometry visual mesh filename=meshes/left_rubber_hand.STL
- link right_rubber_hand: geometry visual mesh filename=meshes/right_rubber_hand.STL
- link torso_primitive_shape: geometry collision box size=0.20 0.31 0.67
Joints:
- joint torso_primitive_shape_joint: origin xyz=0 0 0.15 rpy=0 0 0 -> xyz=0 0 0.14 rpy=0 0 0

File: robot_model/g1_description/g1_29dof_simple_collisions.urdf (robot description, URDF)
Before this commit: robot g1_29dof_lock_waist, 41 links, 40 joints
Joints:
- joint torso_primitive_shape_joint: origin xyz=0 0 0.21 rpy=0 0 0 -> xyz=0 0 0.14 rpy=0 0 0

Commit message: added capsule implementation for mfpp

File: robot_model/g1_description/g1_29dof_lock_waist_modified.urdf (robot description, URDF)
Before this commit: robot g1_29dof_lock_waist, 41 links, 40 joints
Links:
- link torso_primitive_shape: geometry collision cylinder length=0.32 radius=0.11

Commit message: weights used in plan after making tilted stairs wider
also added hands to kin-sca plan and started the robot slightly
backwards

File: robot_model/g1_description/g1_29dof_lock_waist_modified.urdf (robot description, URDF)
Before this commit: robot g1_29dof_lock_waist, 41 links, 40 joints
Links:
- link left_rubber_hand: geometry collision sphere radius=0.035; visual mesh filename=meshes/left_rubber_hand.STL
- link right_rubber_hand: geometry collision sphere radius=0.035; visual mesh filename=meshes/right_rubber_hand.STL

Commit message: preparing code for ral submission
* added ellipsoid-to-ellipsoid collision avoidance
* added more links to fine collision avoidance
* save solve times
* use two separate robot models for kin and dyn planning
* added pelvis to collision model

File: robot_model/g1_description/g1_29dof_lock_waist_modified.urdf (robot description, URDF)
Before this commit: robot g1_29dof_lock_waist, 41 links, 40 joints
Links:
- link left_rubber_hand: geometry visual mesh filename=meshes/left_rubber_hand.STL
- link right_rubber_hand: geometry visual mesh filename=meshes/right_rubber_hand.STL
- link torso_primitive_shape: geometry collision cylinder length=0.46 radius=0.13
Joints:
- joint torso_primitive_shape_joint: origin xyz=0 0 0.14 rpy=0 0 0 -> xyz=0 0 0.11 rpy=0 0 0

File: robot_model/g1_description/g1_29dof_simple_collisions.urdf (robot description, URDF)
Before this commit: robot g1_29dof_lock_waist, 41 links, 40 joints
Links:
- link left_hip_roll_link: geometry collision cylinder length=0.2 radius=0.05; visual mesh filename=meshes/left_hip_roll_link.STL
- link pelvis_contour_link: geometry collision box size=0.1 0.12 0.1; visual mesh filename=meshes/pelvis_contour_link.STL
- link right_hip_roll_link: geometry collision cylinder length=0.2 radius=0.05; visual mesh filename=meshes/right_hip_roll_link.STL
- link torso_primitive_shape: geometry collision cylinder length=0.33 radius=0.11
Joints:
- joint torso_primitive_shape_joint: origin xyz=0 0 0.14 rpy=0 0 0 -> xyz=0 0 0.21 rpy=0 0 0

Commit message: updated files with submission code

File: robot_model/g1_description/g1_29dof_lock_waist_modified.urdf (robot description, URDF)
Before this commit: robot g1_29dof_lock_waist, 41 links, 40 joints
Links:
- link left_rubber_hand: geometry collision sphere radius=0.035; visual sphere radius=0.035
- link right_rubber_hand: geometry collision sphere radius=0.035; visual sphere radius=0.035

File: robot_model/g1_description/g1_29dof_simple_collisions.urdf (robot description, URDF)
Before this commit: robot g1_29dof_simple_collisions, 41 links, 40 joints
Links:
- link left_rubber_hand: geometry collision sphere radius=0.035; visual sphere radius=0.035
- link right_rubber_hand: geometry collision sphere radius=0.035; visual sphere radius=0.035

File: robot_model/ground/navy_door.urdf (robot description, URDF)
Before this commit: robot navy_door, 1 links, 0 joints
Links:
- link door_frame: geometry collision box size=0.518 0.05 2.2; collision box size=0.518 0.05 2.2

File: robot_model/ground/navy_door_fixed.urdf (robot description, URDF)
Before this commit: robot navy_door, 1 links, 0 joints
Links:
- link door_frame: geometry collision box size=0.518 0.05 2.2; collision box size=0.518 0.05 2.2
